File: src/issue3b.kicad_pcb (KiCad board)
At the start: 2 copper layers, 213.1 x 129 mm, 128 parts, among them T1 Coil, X1 14Mhz, X2 4.43Mhz

Commit message: name change
Parts:
- moved LS1 111.7 mm to (233.9, 141.2)
- moved T1 92.5 mm to (241.7, 58.6)
- moved TV1 70.1 mm to (70.2, 43.0)
Routing:
- net Net-(T1-AB): track 59.2 -> 590.0 mm, vias 3 -> 29
- net (no net): track 14361.0 -> 13941.9 mm, vias 827 -> 805
- net +9V: track 517.9 -> 406.0 mm, vias 16 -> 12
Other:
- board text added: "Bambelweeny57"
- board text removed: "Bambleweeny57"

Commit message: Major updates thanks to Liveboxandy and Dee. Some rework from Bambelweeny57.
Parts:
- removed EAR, MIC: Barrel_Jack, spectrum3b:Audio-Connector
- added C25: 22uF, Mod:CP_Axial_L11.0mm_D6.0mm_P20.00mm_Horizontal, F.Cu at (49.8, 98.4)
- added C27: 1uF, Mod:CP_Axial_L11.0mm_D6.0mm_P20.00mm_Horizontal, F.Cu at (204.3, 96.4)
- added C28: 22uF, Mod:CP_Axial_L11.0mm_D6.0mm_P20.32mm_Horizontal, F.Cu at (131.1, 88.8)
- added C34: 22uF, Mod:CP_Axial_L11.0mm_D6.0mm_P20.32mm_Horizontal, F.Cu at (225.3, 69.5)
- added C46: 1uF, Mod:CP_Axial_L11.0mm_D6.0mm_P20.32mm_Horizontal, F.Cu at (225.3, 98.2)
- added C47: 22uF, Mod:CP_Axial_L11.0mm_D6.0mm_P20.32mm_Horizontal, F.Cu at (202.1, 122.8)
- added C50: 22uF, Mod:CP_Axial_L11.0mm_D6.0mm_P20.32mm_Horizontal, F.Cu at (225.3, 76.1)
- added C54: 470pF, Mod:C_Axial_L3.8mm_D2.6mm_P12.70mm_Horizontal, F.Cu at (225.2, 128.5)
- added C65: 22uF, Mod:CP_Axial_L11.0mm_D6.0mm_P20.32mm_Horizontal, F.Cu at (49.8, 95.9)
- added C74: 4.7uF, Mod:CP_Axial_L11.0mm_D6.0mm_P20.32mm_Horizontal, F.Cu at (225.3, 106.8)
- added D1: 1N4148, Mod:D_DO-35_SOD27_P12.70mm_Horizontal, F.Cu at (222.9, 90.4)
- added D11: 1N4148, Mod:D_DO-35_SOD27_P12.70mm_Horizontal, F.Cu at (238.1, 91.2)
- added D12: 1N4148, Mod:D_DO-35_SOD27_P12.70mm_Horizontal, F.Cu at (238.1, 102.5)
- added D13: 1N4148, Mod:D_DO-35_SOD27_P12.40mm_Horizontal, F.Cu at (104.4, 39.5)
- added D15: BA157, Mod:D_DO-35_SOD27_P12.70mm_Horizontal, F.Cu at (238.0, 120.3)
- added D16: BZX85C5V1, Mod:D_DO-35_SOD27_P12.70mm_Horizontal, F.Cu at (238.1, 86.1)
- added D2: 1N4148, Mod:D_DO-35_SOD27_P12.70mm_Horizontal, F.Cu at (222.9, 93.1)
- added D3: 1N4148, Mod:D_DO-35_SOD27_P12.70mm_Horizontal, F.Cu at (222.9, 95.6)
- added D4: 1N4148, Mod:D_DO-35_SOD27_P12.70mm_Horizontal, F.Cu at (222.9, 98.2)
- added D5: 1N4148, Mod:D_DO-35_SOD27_P12.70mm_Horizontal, F.Cu at (222.9, 100.7)
- added D6: 1N4148, Mod:D_DO-35_SOD27_P12.70mm_Horizontal, F.Cu at (222.9, 103.3)
- added D7: 1N4148, Mod:D_DO-35_SOD27_P12.70mm_Horizontal, F.Cu at (222.9, 105.8)
- added D8: 1N4148, Mod:D_DO-35_SOD27_P12.70mm_Horizontal, F.Cu at (222.9, 108.3)
- added D9: 1N4148, Mod:D_DO-35_SOD27_P12.70mm_Horizontal, F.Cu at (222.6, 130.5)
- added E1: Edge_Connector, Mod:Edge Connector, F.Cu at (166.7, 36.4)
- added EAR1: EAR1, Mod:3.5mm_socket, F.Cu at (102.0, 36.0)
- added IC1: ULA, Mod:DIP-40_W15.24mm_Socket, F.Cu at (111.0, 65.9)
- added IC10: 4116, Mod:DIP-16_W7.62mm_Socket, F.Cu at (80.4, 125.6)
- added IC11: 4116, Mod:DIP-16_W7.62mm_Socket, F.Cu at (70.2, 125.6)
- added IC12: 4116, Mod:DIP-16_W7.62mm_Socket, F.Cu at (60.0, 125.6)
- added IC13: 4116, Mod:DIP-16_W7.62mm_Socket, F.Cu at (49.8, 125.7)
- added IC14: LM1889, Mod:DIP-18_W7.62mm_Socket, F.Cu at (69.6, 71.0)
- added IC15: 4532, Mod:DIP-16_W7.62mm_Socket, F.Cu at (186.0, 125.6)
- added IC16: 4532, Mod:DIP-16_W7.62mm_Socket, F.Cu at (175.8, 125.6)
- added IC17: 4532, Mod:DIP-16_W7.62mm_Socket, F.Cu at (165.7, 125.6)
- added IC18: 4532, Mod:DIP-16_W7.62mm_Socket, F.Cu at (155.2, 125.6)
- added IC19: 4532, Mod:DIP-16_W7.62mm_Socket, F.Cu at (191.1, 97.7)
- added IC2: Z80, Mod:DIP-40_W15.24mm_Socket, F.Cu at (183.4, 43.1)
- added IC20: 4532, Mod:DIP-16_W7.62mm_Socket, F.Cu at (180.9, 97.7)
- added IC21: 4532, Mod:DIP-16_W7.62mm_Socket, F.Cu at (170.7, 97.7)
- added IC22: 4532, Mod:DIP-16_W7.62mm_Socket, F.Cu at (160.6, 97.7)
- added IC23: LS32, Mod:DIP-14_W7.62mm_Socket, F.Cu at (168.2, 68.5)
- added IC24: LS00, Mod:DIP-14_W7.62mm_Socket, F.Cu at (153.0, 68.5)
- added IC25: LS157, Mod:DIP-16_W7.62mm_Socket, F.Cu at (139.5, 68.5)
- added IC26: LS157, Mod:DIP-16_W7.62mm_Socket, F.Cu at (168.2, 43.1)
- added IC3: LS157, Mod:DIP-16_W7.62mm_Socket, F.Cu at (137.8, 43.1)
- added IC4: LS157, Mod:DIP-16_W7.62mm_Socket, F.Cu at (152.7, 43.1)
- added IC5: ROM, Mod:DIP-28_W15.24mm_Socket, F.Cu at (206.3, 43.1)
- added IC6: 4116, Mod:DIP-16_W7.62mm_Socket, F.Cu at (121.2, 125.6)
- added IC7: 4116, Mod:DIP-16_W7.62mm_Socket, F.Cu at (111.0, 125.6)
- added IC8: 4116, Mod:DIP-16_W7.62mm_Socket, F.Cu at (100.8, 125.6)
- added IC9: 4116, Mod:DIP-16_W7.62mm_Socket, F.Cu at (90.6, 125.6)
- added J7: Barrel_Jack_MountingPin, Mod:BarrelJack_Horizontal, F.Cu at (248.6, 37.4)
- added JROM1: JROM, Mod:ROM_WireLink, F.Cu at (240.8, 129.7)
- added KB1: Keyboard5, Mod:Keyboard5, F.Cu at (79.0, 103.0)
- added KB2: Keyboard8, Mod:Keyboard8, F.Cu at (220.3, 114.5)
- added MIC1: MIC1, Mod:3.5mm_socket, F.Cu at (117.0, 36.0)
- added OKI-H1: OKI-H, Mod:Wire_Link_7.62mm, F.Cu at (130.1, 35.1)
- added OKI-L1: OKI-L, Mod:Wire_Link_7.62mm, F.Cu at (130.1, 32.5)
- added OKI1: OKI, Mod:Wire_Link_7.62mm, F.Cu at (141.6, 29.9)
- added R34: 15, Mod:R_Axial_DIN0516_L15.5mm_D5.0mm_P22.60mm_Horizontal, F.Cu at (130.6, 42.0)
- added R57: 330, Mod:R_Yageo_L3.6mm_D1.6mm_P12.70mm_Horizontal, F.Cu at (225.3, 123.4)
- added REG1: L7805, Mod:TO-220-3_Horizontal_TabDown, F.Cu at (253.3, 48.0)
- added TI-3: TI-3, Mod:Wire_Link_7.62mm, F.Cu at (141.6, 32.5)
- added TI-4: TI-4, Mod:Wire_Link_7.62mm, F.Cu at (141.6, 35.1)
- added TI1: TI, Mod:Wire_Link_7.62mm, F.Cu at (130.1, 29.9)
- added TR1: ZTX313, Mod:TO-92Flat, F.Cu at (59.0, 66.1)
- added TR2: ZTX313, Mod:TO-92Flat, F.Cu at (62.6, 66.1)
- added TR3: ZTX313, Mod:TO-92Flat, F.Cu at (85.0, 81.1)
- added TR4: ZTX650, Mod:TO-92Flat, F.Cu at (238.1, 116.6)
- added TR5: ZTX315, Mod:TO-92Flat, F.Cu at (243.1, 111.3)
- added TR6: ZTX313, Mod:TO-92Flat, F.Cu at (164.4, 55.4)
- added TR7: ZTX450, Mod:TO-92Flat, F.Cu at (217.1, 134.2)
- added TR8: BC184, Mod:TR9, F.Cu at (105.7, 78.5)
- added TR9: BC184, Mod:TR9, F.Cu at (98.3, 83.8)
- C1, C2, C26, C29, C3, C30, C33, C37, C38, C39, C4, C40, C41, C42, C43, C48, C49, C5, C52, C53, C55, C56, C57, C58, C59, C6, C60, C61, C62, C63, C64, C66, C67, C68, C69, C7, C70, C71, C72, C73, C75, C76, C77, C8: footprint spectrum3b:Passive -> Mod:C_Axial_L3.8mm_D2.6mm_P12.70mm_Horizontal
- C31, C32, C35: footprint spectrum3b:Passive -> Mod:C_Axial_L3.8mm_D2.6mm_P12.40mm_Horizontal
- C44, C45: footprint spectrum3b:Passive -> Mod:CP_Axial_L11.0mm_D6.0mm_P20.32mm_Horizontal
- LS1: footprint spectrum3b:Speaker -> Mod:Speaker
- R1, R10, R11, R12, R13, R14, R15, R16, R17, R18, R19, R2, R20, R21, R22, R23, R24, R25, R26, R27, R28, R29, R3, R30, R31, R32, R33, R4, R42, R43, R44, R45, R46, R47, R48, R49, R5, R50, R51, R52, R53, R54, R55, R56, R58, R59, R6, R60, R61, R62, R63, R64, R65, R66, R67, R68, R69, R7, R70, R71, R72, R73, R74, R75, R76, R77, R78, R8, R9: footprint spectrum3b:Passive -> Mod:R_Yageo_L3.6mm_D1.6mm_P12.70mm_Horizontal
- R35, R36, R37: footprint spectrum3b:Passive -> Mod:R_Yageo_L3.6mm_D1.6mm_P12.40mm_Horizontal
- T1: value Coil -> Transformer_1P_1S; footprint spectrum3b:Coil -> Mod:Coil
- TV1: value Modulator -> TV; footprint spectrum3b:Modulator -> Mod:Modulator
- X1: footprint spectrum3b:X1 -> Mod:X1
- X2: footprint spectrum3b:X2 -> Mod:X2
- moved C43 368.7 mm to (240.7, 86.2)
- moved C66 353.0 mm to (240.7, 81.1)
- moved C49 348.7 mm to (225.5, 83.6)
- moved C41 337.9 mm to (212.1, 39.3)
- moved C61 332.3 mm to (198.7, 147.8)
- moved C77 330.9 mm to (225.5, 81.1)
- moved C57 322.0 mm to (192.3, 119.7)
- moved C62 316.5 mm to (183.4, 147.8)
- moved R33 314.8 mm to (225.3, 126.0)
- moved C55 314.6 mm to (168.2, 147.8)
- moved R54 313.8 mm to (240.7, 102.5)
- moved R58 308.9 mm to (240.7, 91.2)
- moved R26 308.6 mm to (210.0, 125.4)
- moved R59 308.6 mm to (240.7, 93.8)
- moved R27 308.1 mm to (210.0, 128.0)
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Connections:
- C1 pad 1: -5V -> GND
- C1 pad 2: GND -> -5V
- C2 pad 1: -5V -> GND
- C2 pad 2: GND -> -5V
- C3 pad 1: -5V -> GND
- C3 pad 2: GND -> -5V
- C32 pad 1: Net-(D13-K) -> Net-(C32-Pad1)
- C32 pad 2: Net-(C32-Pad2) -> Net-(D13-K)
- C33 pad 1: GND -> +12VA
- C33 pad 2: +12VA -> GND
- C4 pad 1: -5V -> GND
- C4 pad 2: GND -> -5V
- C43 pad 1: GND -> Net-(C43-Pad1)
- C43 pad 2: Net-(C43-Pad2) -> GND
- C48 pad 1: GND -> +12VA
- C48 pad 2: +12VA -> GND
- C49 pad 1: GND -> -12VAC
- C49 pad 2: -12VAC -> GND
- C52 pad 1: Net-(IC14-B-Y_INPUT) -> +12VA
- C52 pad 2: +12VA -> Net-(IC14-B-Y_INPUT)
- C53 pad 1: Net-(IC14-R-Y_INPUT) -> +12VA
- C53 pad 2: +12VA -> Net-(IC14-R-Y_INPUT)
- C55 pad 1: GND -> +5V
- C55 pad 2: +5V -> GND
- C56 pad 1: GND -> +5V
- C56 pad 2: +5V -> GND
- C57 pad 1: GND -> +5V
- C57 pad 2: +5V -> GND
- C58 pad 1: GND -> +5V
- C58 pad 2: +5V -> GND
- C61 pad 1: GND -> +5V
- C61 pad 2: +5V -> GND
- C62 pad 1: GND -> +5V
- C62 pad 2: +5V -> GND
- C66 pad 1: GND -> +9V
- C66 pad 2: +9V -> GND
- C67 pad 1: _CK -> Net-(TR3-B)
- C67 pad 2: Net-(TR3-B) -> _CK
- C77 pad 1: GND -> Net-(T1-AA)
- C77 pad 2: Net-(T1-AA) -> GND
- R1 pad 1: D0 -> Net-(IC1-D0)
- R1 pad 2: Net-(IC1-D0) -> D0
- R11 pad 1: +5V -> D2
- R11 pad 2: D2 -> +5V
- R12 pad 1: +5V -> D3
- R12 pad 2: D3 -> +5V
- R13 pad 1: +5V -> D4
- R13 pad 2: D4 -> +5V
- R14 pad 1: +5V -> D5
- R14 pad 2: D5 -> +5V
- R15 pad 1: +5V -> D6
- R15 pad 2: D6 -> +5V
- R16 pad 1: +5V -> D7
- R16 pad 2: D7 -> +5V
- R17 pad 1: Net-(IC4-2Y) -> /LA0
- R17 pad 2: /LA0 -> Net-(IC4-2Y)
- R18 pad 1: Net-(IC4-1Y) -> /LA1
- R18 pad 2: /LA1 -> Net-(IC4-1Y)
- R19 pad 1: Net-(IC4-4Y) -> /LA2
- R19 pad 2: /LA2 -> Net-(IC4-4Y)
- R2 pad 1: D1 -> Net-(IC1-D1)
- R2 pad 2: Net-(IC1-D1) -> D1
- R20 pad 1: Net-(IC3-3Y) -> /LA3
- R20 pad 2: /LA3 -> Net-(IC3-3Y)
- R21 pad 1: Net-(IC3-2Y) -> /LA4
- R21 pad 2: /LA4 -> Net-(IC3-2Y)
- R22 pad 1: Net-(IC3-1Y) -> /LA5
- R22 pad 2: /LA5 -> Net-(IC3-1Y)
- R23 pad 1: Net-(IC3-4Y) -> /LA6
- R23 pad 2: /LA6 -> Net-(IC3-4Y)
- R25 pad 1: +5V -> Net-(IC2-~{CLK})
- R25 pad 2: Net-(IC2-~{CLK}) -> +5V
- R26 pad 1: _INT -> Net-(IC1-_INT)
- R26 pad 2: Net-(IC1-_INT) -> _INT
- R27 pad 1: _IO_REQ -> _IO_RQULA
- R27 pad 2: _IO_RQULA -> _IO_REQ
- R28 pad 1: +5V -> _NMI
- R28 pad 2: _NMI -> +5V
- R29 pad 1: +5V -> _WAIT
- R29 pad 2: _WAIT -> +5V
- R3 pad 1: D2 -> Net-(IC1-D2)
- R3 pad 2: Net-(IC1-D2) -> D2
- R30 pad 1: +5V -> _BUS_REQ
- R30 pad 2: _BUS_REQ -> +5V
- R35 pad 1: Net-(C31-Pad1) -> Net-(D13-K)
- R35 pad 2: Net-(D13-K) -> Net-(C31-Pad1)
- R36 pad 2: Net-(C32-Pad2) -> Net-(C32-Pad1)
- R4 pad 1: D3 -> Net-(IC1-D3)
- R4 pad 2: Net-(IC1-D3) -> D3
- R43 pad 1: GND -> Net-(IC14-CHROMA_OSC_OUTPUT)
- R43 pad 2: Net-(IC14-CHROMA_OSC_OUTPUT) -> GND
- R44 pad 1: Net-(C72-Pad1) -> Net-(IC14-CHROMA_OSC_OUTPUT)
- R44 pad 2: Net-(IC14-CHROMA_OSC_OUTPUT) -> Net-(C72-Pad1)
- R45 pad 1: Net-(C38-Pad2) -> Net-(IC14-CHROMA_LAG)
- R45 pad 2: Net-(IC14-CHROMA_LAG) -> Net-(C38-Pad2)
- R46 pad 1: GND -> Net-(C38-Pad1)
- R46 pad 2: Net-(C38-Pad1) -> GND
- R48 pad 1: Net-(TR1-B) -> Y
- R48 pad 2: Y -> Net-(TR1-B)
- R49 pad 1: Net-(TR1-B) -> Net-(TR2-C)
- R49 pad 2: Net-(TR2-C) -> Net-(TR1-B)
- R5 pad 1: D4 -> Net-(IC1-D4)
- R5 pad 2: Net-(IC1-D4) -> D4
- R50 pad 1: GND -> Net-(TR1-B)
- R50 pad 2: Net-(TR1-B) -> GND
- R51 pad 1: Net-(TR1-C) -> Net-(TR2-C)
- R51 pad 2: Net-(TR2-C) -> Net-(TR1-C)
- R52 pad 1: GND -> Net-(TR1-E)
- R52 pad 2: Net-(TR1-E) -> GND
- R53 pad 1: GND -> VIDEO
- R53 pad 2: VIDEO -> GND
- R56 pad 1: U -> GND
- R56 pad 2: GND -> U
- R6 pad 1: D5 -> Net-(IC1-D5)
- R6 pad 2: Net-(IC1-D5) -> D5
- R60 pad 1: Net-(TR5-C) -> Net-(C43-Pad1)
- R60 pad 2: Net-(C43-Pad2) -> Net-(TR5-C)
- R61 pad 1: Net-(C43-Pad2) -> Net-(C43-Pad1)
- R62 pad 1: +12V -> +12VA
- R62 pad 2: +12VA -> +12V
- R63 pad 1: V -> GND
- R63 pad 2: GND -> V
- R7 pad 1: D6 -> Net-(IC1-D6)
- R7 pad 2: Net-(IC1-D6) -> D6
- R70 pad 1: Net-(IC25-S) -> Net-(C64-Pad1)
- R70 pad 2: Net-(C64-Pad1) -> Net-(IC25-S)
- R71 pad 1: /_URAS -> Net-(C63-Pad1)
- R71 pad 2: Net-(C63-Pad1) -> /_URAS
- R73 pad 1: +5V -> _CK
- R73 pad 2: _CK -> +5V
- R76 pad 1: Net-(TR9-C) -> Net-(IC14-B-Y_INPUT)
- R76 pad 2: Net-(IC14-B-Y_INPUT) -> Net-(TR9-C)
- R77 pad 1: Net-(TR8-C) -> Net-(IC14-R-Y_INPUT)
- R77 pad 2: Net-(IC14-R-Y_INPUT) -> Net-(TR8-C)
- R78 pad 1: +5V -> Net-(IC14-CHROMA_BIAS)
- R78 pad 2: Net-(IC14-CHROMA_BIAS) -> +5V
- R8 pad 1: D7 -> Net-(IC1-D7)
- R8 pad 2: Net-(IC1-D7) -> D7
- T1 pad 5: (no net) -> unconnected-(T1-Pad5)
- T1 pad 6: (no net) -> unconnected-(T1-Pad6)
Routing:
- net (no net): track 13941.9 -> 111.9 mm, vias 805 -> 0
- net +5V: track 1868.5 -> 1173.4 mm, vias 146 -> 32
- net Net-(TR8-C): track 584.1 -> 41.9 mm, vias 31 -> 2
- net Net-(T1-AB): track 590.0 -> 59.2 mm, vias 29 -> 1
- net +12VA: track 0.00 -> 430.1 mm, vias 0 -> 6
- net +12V: track 0.00 -> 419.0 mm, vias 0 -> 5
- net /_LRAS: track 0.00 -> 361.5 mm, vias 0 -> 8
- net A15: track 0.00 -> 351.5 mm, vias 0 -> 10
- net A14: track 0.00 -> 286.4 mm, vias 0 -> 6
- net Net-(IC14-R-Y_INPUT): track 363.0 -> 77.5 mm, vias 19 -> 1
- net _IO_RQULA: track 0.00 -> 282.6 mm, vias 0 -> 6
- net _M_REQ: track 0.00 -> 272.4 mm, vias 0 -> 6
- net D0: track 0.00 -> 262.7 mm, vias 0 -> 8
- net _RD: track 0.00 -> 259.6 mm, vias 0 -> 5
- net Y: track 0.00 -> 259.3 mm, vias 0 -> 4
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Other:
- outline, holes or cut-outs redrawn
- board text added: "Bambelweeny57 - Liveboxandy - Dee"
- board text removed: "Bambelweeny57"
