File: src/issue3b.kicad_sch (KiCad schematic)
At the start: 199 parts, among them IC1 ULA, IC10 4116, IC11 4116, IC12 4116, IC13 4116, IC14 LM1889, IC15 4532, IC16 4532, IC17 4532, IC18 4532, IC19 4532, IC2 Z80, IC20 4532, IC21 4532, IC22 4532, IC23 74LS32, IC24 74LS00, IC25 74LS157, IC26 74LS157, IC3 LS157, IC4 LS157, IC5 ROM, IC6 4116, IC7 4116, IC8 4116, IC9 4116, J7 Barrel_Jack_MountingPin, T1 Coil, X1 14Mhz, X2 4.43Mhz

Commit message: changed to kicad 10 and added bljall-alt 3d models.
Parts:
- EAR1: renamed from Ear0; footprint (none) -> spectrum3b:Audio-Connector
- MIC1: renamed from Mic0; footprint (none) -> spectrum3b:Audio-Connector

Commit message: Major updates thanks to Liveboxandy and Dee. Some rework from Bambelweeny57.
Parts:
- added BM1, LL1, LR1, TM1: MountingHole, Mod:MountingHole_3.3mm Spectrum, symbol Mechanical:MountingHole
- added C54: 470pF, Mod:C_Axial_L3.8mm_D2.6mm_P12.70mm_Horizontal, symbol Device:C
- added LM1, RM1, RM2: MountingHole, Mod:MountingHole_5mm Spectrum, symbol Mechanical:MountingHole
- added R57: 330, Mod:R_Yageo_L3.6mm_D1.6mm_P12.70mm_Horizontal, symbol Device:R
- C1, C2, C26, C29, C3, C30, C33, C37, C38, C39, C4, C40, C41, C42, C43, C48, C49, C5, C52, C53, C55, C56, C57, C58, C59, C6, C60, C61, C62, C63, C64, C66, C67, C68, C69, C7, C70, C71, C72, C73, C75, C76, C77, C8: footprint spectrum3b:Passive -> Mod:C_Axial_L3.8mm_D2.6mm_P12.70mm_Horizontal
- C25, C27: footprint (none) -> Mod:CP_Axial_L11.0mm_D6.0mm_P20.00mm_Horizontal
- C28, C34, C46, C47, C50, C65, C74: footprint (none) -> Mod:CP_Axial_L11.0mm_D6.0mm_P20.32mm_Horizontal
- C31, C32, C35: footprint spectrum3b:Passive -> Mod:C_Axial_L3.8mm_D2.6mm_P12.40mm_Horizontal
- C44, C45: footprint spectrum3b:Passive -> Mod:CP_Axial_L11.0mm_D6.0mm_P20.32mm_Horizontal
- D1, D11, D12, D15, D2, D3, D4, D5, D6, D7, D8, D9: footprint (none) -> Mod:D_DO-35_SOD27_P12.70mm_Horizontal
- D13: footprint (none) -> Mod:D_DO-35_SOD27_P12.40mm_Horizontal
- D16: value DZY88 -> BZX85C5V1; footprint (none) -> Mod:D_DO-35_SOD27_P12.70mm_Horizontal
- E1: footprint (none) -> Mod:Edge Connector
- EAR1: value Barrel_Jack -> EAR1; footprint spectrum3b:Audio-Connector -> Mod:3.5mm_socket
- IC1, IC2: footprint (none) -> Mod:DIP-40_W15.24mm_Socket
- IC10, IC11, IC12, IC13, IC15, IC16, IC17, IC18, IC19, IC20, IC21, IC22, IC3, IC4, IC6, IC7, IC8, IC9: footprint (none) -> Mod:DIP-16_W7.62mm_Socket
- IC14: footprint (none) -> Mod:DIP-18_W7.62mm_Socket
- IC23: value 74LS32 -> LS32; footprint (none) -> Mod:DIP-14_W7.62mm_Socket
- IC24: value 74LS00 -> LS00; footprint (none) -> Mod:DIP-14_W7.62mm_Socket
- IC25, IC26: value 74LS157 -> LS157; footprint (none) -> Mod:DIP-16_W7.62mm_Socket
- IC5: footprint (none) -> Mod:DIP-28_W15.24mm_Socket
- J7: footprint (none) -> Mod:BarrelJack_Horizontal
- JROM1: footprint (none) -> Mod:ROM_WireLink
- KB1: value Conn_01x05 -> Keyboard5; footprint (none) -> Mod:Keyboard5; symbol Connector_Generic:Conn_01x05 -> ZXSpectrumIssue3B:Keyboard5
- KB2: value Conn_01x08 -> Keyboard8; footprint (none) -> Mod:Keyboard8; symbol Connector_Generic:Conn_01x08 -> ZXSpectrumIssue3B:Keyboard8
- LS1: footprint spectrum3b:Speaker -> Mod:Speaker
- MIC1: value Barrel_Jack -> MIC1; footprint spectrum3b:Audio-Connector -> Mod:3.5mm_socket
- OKI-H1, OKI-L1, OKI1, TI-3, TI-4, TI1: footprint (none) -> Mod:Wire_Link_7.62mm
- R1, R10, R11, R12, R13, R14, R15, R16, R17, R18, R19, R2, R20, R21, R22, R23, R24, R25, R26, R27, R28, R29, R3, R30, R31, R32, R33, R4, R42, R43, R44, R45, R46, R47, R48, R49, R5, R50, R51, R52, R53, R54, R55, R56, R58, R59, R6, R60, R61, R62, R63, R64, R65, R66, R67, R68, R69, R7, R70, R71, R72, R73, R74, R75, R76, R77, R78, R8, R9: footprint spectrum3b:Passive -> Mod:R_Yageo_L3.6mm_D1.6mm_P12.70mm_Horizontal
- R34: footprint (none) -> Mod:R_Axial_DIN0516_L15.5mm_D5.0mm_P22.60mm_Horizontal
- R35, R36, R37: footprint spectrum3b:Passive -> Mod:R_Yageo_L3.6mm_D1.6mm_P12.40mm_Horizontal
- REG1: footprint (none) -> Mod:TO-220-3_Horizontal_TabDown
- T1: value Coil -> Transformer_1P_1S; footprint spectrum3b:Coil -> Mod:Coil; symbol Device:Transformer_1P_1S -> ZXSpectrumIssue3B:Transformer_1P_1S
- TR1, TR2, TR3, TR4, TR6, TR7: footprint (none) -> Mod:TO-92Flat
- TR5: value ZTX213 -> ZTX315; footprint (none) -> Mod:TO-92Flat
- TR8, TR9: footprint (none) -> Mod:TR9
- TV1: value Modulator -> TV; footprint spectrum3b:Modulator -> Mod:Modulator
- X1: footprint spectrum3b:X1 -> Mod:X1
- X2: footprint spectrum3b:X2 -> Mod:X2
Connections:
- net +12V: now also R62.2; no longer R62.1
- net +12VA: now also C33.1, C48.1, C52.1, C53.1, R62.1; no longer C33.2, C48.2, C52.2, C53.2, R62.2
- net +5V: now also C55.1, C56.1, C57.1, C58.1, C61.1, C62.1, R11.2, R12.2, R13.2, R14.2, R15.2, R16.2, R25.2, R28.2, R29.2, R30.2, R73.2, R78.2; no longer C55.2, C56.2, C57.2, C58.2, C61.2, C62.2, R11.1, R12.1, R13.1, R14.1, R15.1, R16.1, R25.1, R28.1, R29.1, R30.1, R73.1, R78.1, TR7.1 (C)
- net +9V: now also C66.1, TR7.1 (C); no longer C66.2
- net -12VAC: now also C49.1; no longer C49.2
- net -5V: now also C1.2, C2.2, C3.2, C4.2; no longer C1.1, C2.1, C3.1, C4.1
- net D0: now also R1.2; no longer R1.1
- net D1: now also R2.2; no longer R2.1
- net D2: now also R11.1, R3.2; no longer R11.2, R3.1
- net D3: now also R12.1, R4.2; no longer R12.2, R4.1
- net D4: now also R13.1, R5.2; no longer R13.2, R5.1
- net D5: now also R14.1, R6.2; no longer R14.2, R6.1
- net D6: now also R15.1, R7.2; no longer R15.2, R7.1
- net D7: now also R16.1, R8.2; no longer R16.2, R8.1
- net GND: now also C1.1, C2.1, C3.1, C33.2, C4.1, C43.2, C48.2, C49.2, C55.2, C56.2, C57.2, C58.2, C61.2, C62.2, C66.2, C77.2, R43.2, R46.2, R50.2, R52.2, R53.2, R56.1, R63.1, C54.2; no longer C1.2, C2.2, C3.2, C33.1, C4.2, C43.1, C48.1, C49.1, C55.1, C56.1, C57.1, C58.1, C61.1, C62.1, C66.1, C77.1, R43.1, R46.1, R50.1, R52.1, R53.1, R56.2, R63.2
- net LA0: now also R17.1; no longer R17.2
- net LA1: now also R18.1; no longer R18.2
- net LA2: now also R19.1; no longer R19.2
- net LA3: now also R20.1; no longer R20.2
- net LA4: now also R21.1; no longer R21.2
- net LA5: now also R22.1; no longer R22.2
- net LA6: now also R23.1; no longer R23.2
- net U: now also R56.2; no longer R56.1
- net V: now also R63.2; no longer R63.1
- net VIDEO: now also R53.1; no longer R53.2
- net Y: now also R48.1; no longer R48.2
- net _BUS_REQ: now also R30.1; no longer R30.2
- net _CK: now also C67.2, R73.1; no longer C67.1, R73.2
- net _INT: now also R26.2; no longer R26.1
- net _IO_REQ: now also R27.2; no longer R27.1
- net _IO_RQULA: now also R27.1; no longer R27.2
- net _LRAS: now also R57.1
- net _NMI: now also R28.1; no longer R28.2
- net _RFSH: now also C54.1, R57.2
- net _URAS: now also R71.2; no longer R71.1
- net _WAIT: now also R29.1; no longer R29.2
- net at IC1.12 (_INT): now also R26.1; no longer R26.2
- net at IC1.18 (D0), IC6.14 (DOUT), IC6.2 (DIN): now also R1.1; no longer R1.2
- net at IC1.19 (KB0), KB1.1, R69.2: now also KB1.11 (A1)
- net at IC1.20 (KB1), KB1.2, R68.2: now also KB1.12 (2A)
- net at IC1.21 (D1), IC7.14 (DOUT), IC7.2 (DIN): now also R2.1; no longer R2.2
- net at IC1.22 (D2), IC8.14 (DOUT), IC8.2 (DIN): now also R3.1; no longer R3.2
- net at IC1.23 (KB2), KB1.3, R67.2: now also KB1.13 (3A)
- net at IC1.24 (KB3), KB1.4, R66.2: now also KB1.14 (4A)
- net at IC1.25 (D3), IC9.14 (DOUT), IC9.2 (DIN): now also R4.1; no longer R4.2
- net at IC1.26 (KB4), KB1.5, R65.2: now also KB1.15 (5A)
- net at IC1.27 (D4), IC10.14 (DOUT), IC10.2 (DIN): now also R5.1; no longer R5.2
- net at C35.2, D13.1 (K), D9.2 (A)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: now also C32.2, R35.1; no longer C32.1, R35.2
- net at IC1.29 (D5), IC11.14 (DOUT), IC11.2 (DIN): now also R6.1; no longer R6.2
- net at IC1.30 (D6), IC12.14 (DOUT), IC12.2 (DIN): now also R7.1; no longer R7.2
- net at IC1.31 (D7), IC13.14 (DOUT), IC13.2 (DIN): now also R8.1; no longer R8.2
- net at IC3.12 (4Y): now also R23.2; no longer R23.1
- net at IC3.4 (1Y): now also R22.2; no longer R22.1
- net at IC3.7 (2Y): now also R21.2; no longer R21.1
- net at IC3.9 (3Y): now also R20.2; no longer R20.1
- net at IC4.12 (4Y): now also R19.2; no longer R19.1
- net at IC4.4 (1Y): now also R18.2; no longer R18.1
- net at IC4.7 (2Y): now also R17.2; no longer R17.1
- net at C65.2, TR1.1 (C), TR2.2 (B): now also R51.2; no longer R51.1
- net at IC2.6 (~{CLK}), TR3.1 (C): now also R25.1; no longer R25.2
- net at R24.1, TR3.2 (B): now also C67.1; no longer C67.2
- net at D1.2 (A), KB2.1 (Pin_1): now also KB2.11 (Pin_1A)
- net at D2.2 (A), KB2.2 (Pin_2): now also KB2.12 (Pin_2A)
- net at D3.2 (A), KB2.3 (Pin_3): now also KB2.13 (Pin_3A)
- net at D4.2 (A), KB2.4 (Pin_4): now also KB2.14 (Pin_4A)
- net at D5.2 (A), KB2.5 (Pin_5): now also KB2.15 (Pin_5A)
- net at D6.2 (A), KB2.6 (Pin_6): now also KB2.16 (Pin_6A)
- net at D7.2 (A), KB2.7 (Pin_7): now also KB2.17 (Pin_7A)
- net at D8.2 (A), KB2.8 (Pin_8): now also KB2.18 (Pin_8A)
- net at C25.1, C40.1, C42.1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: now also R49.1, R51.1; no longer R49.2, R51.2
- net at R36.2: now also C32.1; no longer C32.2
- net at C31.1: now also R35.2; no longer R35.1
- net at C37.1, IC14.18 (CHROMA_LAG): now also R45.1; no longer R45.2
- net at C76.2, IC14.3 (CHROMA_BIAS): now also R78.1; no longer R78.2
- net at C71.1, TR8.1 (C): now also R77.2; no longer R77.1
- net at C69.1, TR9.1 (C): now also R76.2; no longer R76.1
- net at C72.1, X2.1: now also R44.2; no longer R44.1
- net at C38.2, X2.2: now also R45.2; no longer R45.1
- net at C38.1, C39.2: now also R46.1; no longer R46.2
- net at TR1.3 (E): now also R52.1; no longer R52.2
- net at IC23.8, IC25.1 (S), IC26.1 (S): now also R70.2; no longer R70.1
- net at C63.1, IC23.9: now also R71.1; no longer R71.2
- net at C64.1, IC23.5: now also R70.1; no longer R70.2
- net at TR5.1 (C): now also R60.2; no longer R60.1
- net at R61.2, T1.1 (AA): now also C77.1; no longer C77.2
- new net: IC14.17 (CHROMA_OSC_OUTPUT), R43.1, R44.1
- new net: C53.2, IC14.2 (R-Y_INPUT), R77.1
- new net: C52.2, IC14.4 (B-Y_INPUT), R76.1
- new net: R48.2, R49.2, R50.1, TR1.2 (B)
- new net: C43.1, R60.1, R61.1
- new net NC: J7.3 (MP2)
- no-connect marks 4 -> 15
Other:
- title: ZX Spectrum -> ZX Spectrum 16K/48K
- moved on the sheet: C1, C2, C3, C32, C33, C4, C43, C48, C49, C52, C53, C55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
